File: hardware/gausCheck_LED.kicad_sch (KiCad schematic)
At the start: 7 parts, among them Q1 BSS138

Commit message: update Mouser Nr..
Parts:
- Q1: Mouser (none) -> 512-BSS138
Changed lines of the file:
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@@
       (effects (font (size 1.27 1.27)) hide)
     )
+    (pin "1")
     (pin "2")
-    (pin "1")
     (instances
       (project "gaussCheck"
@@
       (effects (font (size 1.27 1.27)) hide)
     )
+    (pin "1")
     (pin "2")
-    (pin "1")
     (instances
       (project "gaussCheck"
@@
       (effects (font (size 1.27 1.27)) hide)
     )
-    (pin "3")
+    (property "Mouser" "512-BSS138" (at 128.27 107.95 0)
+      (effects (font (size 1.27 1.27)) hide)
+    )
     (pin "1")
     (pin "2")
+    (pin "3")
     (instances
       (project "gaussCheck"
@@
       (effects (font (size 1.27 1.27)) hide)
     )
+    (pin "1")
     (pin "2")
-    (pin "1")
     (instances
       (project "gaussCheck"
