File: hardware/gausCheck_MCU.kicad_sch (KiCad schematic)
At the start: 21 parts, among them J2 SWD, SW1 PTS810, U3 ATSAML22N18A-AUT, Y1 32.768kHz

Commit message: updated some MPNs
Parts:
- C2, C3: value ??p -> 8p; MPN CC0603JRNPO9BN220 -> CC0603DRNPO9BN8R0; Mouser 603-CC603JRNPO9BN220 -> 603-CC603DRNPO9BN8R0
- C6: MPN (none) -> GRM188R60J106ME84D
- J2: MPN (none) -> BD125-10-A-0305-0580-L-B
- SW1: MPN (none) -> PTS810 SJG 250 SMTR LFS
- U3: MPN (none) -> ATSAML22N18A-AUT
- Y1: MPN (none) -> SC32S-7PF20PPM; Mouser (none) -> 628-SC32S-7PF20PPM
Other:
- note added: "CL=7pF Cstray=4pF C10,C9=8pF [((8x8)/(8+8))+3]"
Changed lines of the file:
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@@
     (stroke (width 0) (type default))
+  )
+  (text "CL=7pF\nCstray=4pF\nC10,C9=8pF [((8x8)/(8+8))+3]" (at 92.71 26.67 0)
+    (effects (font (size 1.27 1.27)) (justify left bottom))
   )
   (label "LED3" (at 247.65 96.52 0) (fields_autoplaced)
@@
     )
     (property "Datasheet" "https://ww1.microchip.com/downloads/aemDocuments/documents/MCU32/ProductDocuments/DataSheets/SAM-L22-Family-Data-Sheet-DS60001465.pdf" (at 142.24 124.46 0)
+      (effects (font (size 1.27 1.27)) hide)
+    )
+    (property "MPN" "ATSAML22N18A-AUT" (at 142.24 68.58 0)
       (effects (font (size 1.27 1.27)) hide)
     )
@@
       (effects (font (size 1.27 1.27)) hide)
     )
+    (property "MPN" "PTS810 SJG 250 SMTR LFS" (at 119.38 171.45 0)
+      (effects (font (size 1.27 1.27)) hide)
+    )
     (pin "1")
     (pin "2")
@@
     )
     (property "Datasheet" "~" (at 146.05 176.53 0)
+      (effects (font (size 1.27 1.27)) hide)
+    )
+    (property "MPN" "BD125-10-A-0305-0580-L-B" (at 146.05 176.53 0)
       (effects (font (size 1.27 1.27)) hide)
     )
@@
       (effects (font (size 1.27 1.27)) hide)
     )
+    (property "MPN" "GRM188R60J106ME84D" (at 27.94 148.59 0)
+      (effects (font (size 1.27 1.27)) hide)
+    )
     (pin "1")
     (pin "2")
@@
     )
     (property "Datasheet" "https://ww1.microchip.com/downloads/aemDocuments/documents/MCU32/ProductDocuments/DataSheets/SAM-L22-Family-Data-Sheet-DS60001465.pdf" (at 62.23 223.52 0)
+      (effects (font (size 1.27 1.27)) hide)
+    )
+    (property "MPN" "ATSAML22N18A-AUT" (at 62.23 167.64 0)
       (effects (font (size 1.27 1.27)) hide)
     )
@@
       (effects (font (size 1.27 1.27)) (justify left))
     )
-    (property "Value" "??p" (at 115.7732 40.767 0)
+    (property "Value" "8p" (at 115.7732 40.767 0)
       (effects (font (size 1.27 1.27)) (justify left))
     )
@@
       (effects (font (size 1.27 1.27)) hide)
     )
-    (property "MPN" "CC0603JRNPO9BN220" (at 118.11 41.91 0)
-      (effects (font (size 1.27 1.27)) hide)
-    )
-    (property "Mouser" "603-CC603JRNPO9BN220 " (at 118.11 41.91 0)
+    (property "MPN" "CC0603DRNPO9BN8R0" (at 118.11 41.91 0)
+      (effects (font (size 1.27 1.27)) hide)
+    )
+    (property "Mouser" "603-CC603DRNPO9BN8R0" (at 118.11 41.91 0)
       (effects (font (size 1.27 1.27)) hide)
     )
@@
       (effects (font (size 1.27 1.27)) (justify left))
     )
-    (property "Value" "??p" (at 104.3432 40.767 0)
+    (property "Value" "8p" (at 104.3432 40.767 0)
       (effects (font (size 1.27 1.27)) (justify left))
     )
@@
       (effects (font (size 1.27 1.27)) hide)
     )
-    (property "Mouser" "603-CC603JRNPO9BN220 " (at 106.68 41.91 0)
-      (effects (font (size 1.27 1.27)) hide)
-    )
-    (property "MPN" "CC0603JRNPO9BN220" (at 106.68 41.91 0)
+    (property "Mouser" "603-CC603DRNPO9BN8R0" (at 106.68 41.91 0)
+      (effects (font (size 1.27 1.27)) hide)
+    )
+    (property "MPN" "CC0603DRNPO9BN8R0" (at 106.68 41.91 0)
       (effects (font (size 1.27 1.27)) hide)
     )
@@
       (effects (font (size 1.27 1.27)) hide)
     )
-    (property "Datasheet" "~" (at 111.76 33.02 0)
+    (property "Datasheet" "https://www.mouser.de/datasheet/2/360/file_PRODUCT_MASTER_50812_GRAPHIC03-542305.pdf" (at 111.76 33.02 0)
+      (effects (font (size 1.27 1.27)) hide)
+    )
+    (property "MPN" "SC32S-7PF20PPM" (at 111.76 33.02 0)
+      (effects (font (size 1.27 1.27)) hide)
+    )
+    (property "Mouser" "628-SC32S-7PF20PPM" (at 111.76 33.02 0)
       (effects (font (size 1.27 1.27)) hide)
     )
@@
     )
     (property "Datasheet" "https://ww1.microchip.com/downloads/aemDocuments/documents/MCU32/ProductDocuments/DataSheets/SAM-L22-Family-Data-Sheet-DS60001465.pdf" (at 224.79 99.06 0)
+      (effects (font (size 1.27 1.27)) hide)
+    )
+    (property "MPN" "ATSAML22N18A-AUT" (at 224.79 68.58 0)
       (effects (font (size 1.27 1.27)) hide)
     )
@@
       (effects (font (size 1.27 1.27)) hide)
     )
+    (property "MPN" "ATSAML22N18A-AUT" (at 59.69 68.58 0)
+      (effects (font (size 1.27 1.27)) hide)
+    )

Commit message: custom LED daughter board for display lightning added resistors to USB-C CC line
Connections:
- net EN_DisplayLED: now reaches U3.67 (PB19/SLCD[45])
- no-connect marks 29 -> 28
Changed lines of the file:
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@@
   (no_connect (at 165.1 83.82))
   (no_connect (at 165.1 88.9))
-  (no_connect (at 247.65 83.82))
   (no_connect (at 247.65 76.2))
   (no_connect (at 165.1 73.66))
@@
   (no_connect (at 140.97 179.07))
   (no_connect (at 165.1 81.28))
-  (no_connect (at 165.1 78.74))
+  (no_connect (at 247.65 83.82))
   (no_connect (at 247.65 81.28))
   (no_connect (at 165.1 71.12))
@@
     (stroke (width 0) (type default))
   )
+  (wire (pts (xy 165.1 78.74) (xy 184.15 78.74))
+    (stroke (width 0) (type default))
+  )
   (wire (pts (xy 36.83 151.13) (xy 36.83 152.4))
     (stroke (width 0) (type default))
@@
   )
   (hierarchical_label "Sense_VBat" (shape input) (at 261.62 35.56 0) (fields_autoplaced)
+    (effects (font (size 1.27 1.27)) (justify left))
+  )
+  (hierarchical_label "EN_DisplayLED" (shape output) (at 184.15 78.74 0) (fields_autoplaced)
     (effects (font (size 1.27 1.27)) (justify left))
   )
@@
     (pin "16")
     (pin "9")
-    (pin "3")
     (pin "33")
     (pin "34")
@@
     (pin "24")
     (pin "25")
+    (pin "3")
     (instances
       (project "gaussCheck"

Commit message: update Mouser Nr..
Parts:
- C12, C4, C5, C7: MPN (none) -> C0603C104K9RACTU; Mouser (none) -> 80-C0603C104K9R
- C3, C8: MPN (none) -> C0603C105Z9VACTU; Mouser (none) -> 80-C0603C105Z9V
- C6: MPN GRM188R60J106ME84D -> C1608X5R0J106K080AB; Mouser (none) -> 810-C1608X5R0J106K
- J2: Mouser (none) -> 640-BD12510A305580LB
- L2: Mouser (none) -> 810-MLZ2012M100HT000
- R1: MPN (none) -> CRCW06031K00FKEA; Mouser (none) -> 71-CRCW0603-1.0K-E3
- R2: MPN (none) -> CRCW060310K0FKEI; Mouser (none) -> 71-CRCW060310K0FKEI
- R3: MPN (none) -> CRCW0603300RFKEAC; Mouser (none) -> 71-CRCW0603300RFKEAC
- SW1: Mouser (none) -> 611-PTS810SJG250SMTR
- U3: Mouser (none) -> 556-ATSAML22N18A-AUT

Commit message: change debug connector..
Parts:
- J2: MPN BD125-10-A-0305-0580-L-B -> 1156861; Mouser 640-BD12510A305580LB -> 651-1156861
Changed lines of the file:
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@@
       (effects (font (size 1.27 1.27)) hide)
     )
-    (property "MPN" "BD125-10-A-0305-0580-L-B" (at 146.05 176.53 0)
+    (property "MPN" "1156861" (at 146.05 176.53 0)
       (effects (font (size 1.27 1.27)) hide)
     )
-    (property "Mouser" "640-BD12510A305580LB" (at 146.05 176.53 0)
+    (property "Mouser" "651-1156861" (at 146.05 176.53 0)
       (effects (font (size 1.27 1.27)) hide)
     )
